Commit message: updated the comments for urdf and the mobile links

File: src/uncertainty-nav/urdf/turtlebot3_waffle_pi_uncertainty.urdf.xacro (robot description, xacro)
@@ -1,3 +1,17 @@
 <?xml version="1.0" ?>
+<!--
+  TurtleBot3 Waffle Pi — Gazebo URDF with real LDS-01 laser sensor.
+  This file extends the official turtlebot3_description URDF by:
+    1. Keeping the exact TurtleBot3 Waffle Pi geometry and inertia
+    2. Using the real LDS-01 sensor spec:
+         - 360 samples per scan
+         - 360° FoV (0 to 2π)
+         - Range: 0.12 m to 3.5 m
+         - Update rate: 5 Hz (real hardware) — set to 10 Hz for sim
+    3. Making laser noise std configurable via xacro argument
+       so Env A (std=0.01) and Env B (std=0.05) use the same URDF
+  Usage in launch file:
+    xacro turtlebot3_waffle_pi_uncertainty.urdf.xacro laser_noise_std:=0.01
+-->
 <robot name="turtlebot3_waffle_pi" xmlns:xacro="http://ros.org/wiki/xacro">
   <!-- ── Configurable parameters ──────────────────────────────────────── -->
@@ -41,4 +55,81 @@
     </inertial>
   </link>
+  <!-- ── Wheel joints and links ────────────────────────────────────────── -->
+  <joint name="wheel_left_joint" type="continuous">
+    <parent link="base_link"/>
+    <child link="wheel_left_link"/>
+    <origin xyz="0.0 0.144 0.023" rpy="-1.57079632679 0 0"/>
+    <axis xyz="0 0 1"/>
+  </joint>
+  <link name="wheel_left_link">
+    <visual>
+      <origin xyz="0 0 0" rpy="1.57079632679 0 0"/>
+      <geometry><mesh filename="package://turtlebot3_description/meshes/wheels/left_tire.stl" scale="0.001 0.001 0.001"/></geometry>
+      <material name="dark"/>
+    </visual>
+    <collision>
+      <origin xyz="0 0 0" rpy="0 0 0"/>
+      <geometry><cylinder length="0.018" radius="0.033"/></geometry>
+    </collision>
+    <inertial>
+      <origin xyz="0 0 0" rpy="0 0 0"/>
+      <mass value="0.02844"/>
+      <inertia ixx="1.1175580e-05" ixy="-4.2369783e-11" ixz="-5.9381719e-09"
+               iyy="1.1192413e-05" iyz="-1.4400107e-11" izz="2.0712558e-05"/>
+    </inertial>
+  </link>
+  <joint name="wheel_right_joint" type="continuous">
+    <parent link="base_link"/>
+    <child link="wheel_right_link"/>
+    <origin xyz="0.0 -0.144 0.023" rpy="-1.57079632679 0 0"/>
+    <axis xyz="0 0 1"/>
+  </joint>
+  <link name="wheel_right_link">
+    <visual>
+      <origin xyz="0 0 0" rpy="1.57079632679 0 0"/>
+      <geometry><mesh filename="package://turtlebot3_description/meshes/wheels/right_tire.stl" scale="0.001 0.001 0.001"/></geometry>
+      <material name="dark"/>
+    </visual>
+    <collision>
+      <origin xyz="0 0 0" rpy="0 0 0"/>
+      <geometry><cylinder length="0.018" radius="0.033"/></geometry>
+    </collision>
+    <inertial>
+      <origin xyz="0 0 0" rpy="0 0 0"/>
+      <mass value="0.02844"/>
+      <inertia ixx="1.1175580e-05" ixy="-4.2369783e-11" ixz="-5.9381719e-09"
+               iyy="1.1192413e-05" iyz="-1.4400107e-11" izz="2.0712558e-05"/>
+    </inertial>
+  </link>
+  <!-- ── Caster wheel ───────────────────────────────────────────────────── -->
+  <joint name="caster_back_right_joint" type="fixed">
+    <parent link="base_link"/>
+    <child link="caster_back_right_link"/>
+    <origin xyz="-0.177 -0.064 -0.004" rpy="-1.57079632679 0 0"/>
+  </joint>
+  <link name="caster_back_right_link">
+    <collision><origin xyz="0 0.001 0" rpy="0 0 0"/>
+      <geometry><sphere radius="0.018"/></geometry></collision>
+    <inertial><origin xyz="0 0 0" rpy="0 0 0"/><mass value="0.005"/>
+      <inertia ixx="3.6e-07" ixy="0" ixz="0" iyy="3.6e-07" iyz="0" izz="3.6e-07"/></inertial>
+  </link>
+  <joint name="caster_back_left_joint" type="fixed">
+    <parent link="base_link"/>
+    <child link="caster_back_left_link"/>
+    <origin xyz="-0.177 0.064 -0.004" rpy="-1.57079632679 0 0"/>
+  </joint>
+  <link name="caster_back_left_link">
+    <collision><origin xyz="0 0.001 0" rpy="0 0 0"/>
+      <geometry><sphere radius="0.018"/></geometry></collision>
+    <inertial><origin xyz="0 0 0" rpy="0 0 0"/><mass value="0.005"/>
+      <inertia ixx="3.6e-07" ixy="0" ixz="0" iyy="3.6e-07" iyz="0" izz="3.6e-07"/></inertial>
+  </link>
+  <!-- ── IMU link ───────────────────────────────────────────────────────── -->
+  <joint name="imu_joint" type="fixed">
+    <parent link="base_link"/>
+    <child link="imu_link"/>
+    <origin xyz="-0.032 0 0.068" rpy="0 0 0"/>
+  </joint>
+  <link name="imu_link"/>
   <!-- ── LDS-01 laser scanner ───────────────────────────────────────────── -->
   <!--
